Commit message: urdf change

File: HW/urdf/urdf/HEXAPEDAL_URDF.xacro (robot description, xacro)
@@ -406,5 +406,5 @@
 <link name="RB_flame4_1">
   <inertial>
-    <origin xyz="-0.020163841378835465 0.020163841393334644 -0.003624618500374904" rpy="0 0 0"/>
+    <origin xyz="-0.020163841378833314 0.02016384139333624 -0.0036246185003608977" rpy="0 0 0"/>
     <mass value="0.06395081687871436"/>
     <inertia ixx="6.2e-05" iyy="6.2e-05" izz="7.4e-05" ixy="1.7e-05" iyz="2e-06" ixz="-2e-06"/>
@@ -506,5 +506,5 @@
 <link name="LF_flame4_1">
   <inertial>
-    <origin xyz="0.020163841378832717 -0.020163841393343346 -0.0036246185003829686" rpy="0 0 0"/>
+    <origin xyz="0.020163841378835992 -0.020163841393339085 -0.003624618500361524" rpy="0 0 0"/>
     <mass value="0.06395081687871436"/>
     <inertia ixx="6.2e-05" iyy="6.2e-05" izz="7.4e-05" ixy="1.7e-05" iyz="-2e-06" ixz="2e-06"/>
@@ -526,5 +526,5 @@
 <link name="RF_DS51150_270_1_1">
   <inertial>
-    <origin xyz="-0.02303277026668618 -0.023032770253798768 -0.006733285359171658" rpy="0 0 0"/>
+    <origin xyz="-0.023032770266679756 -0.023032770253798393 -0.0067332853591638014" rpy="0 0 0"/>
     <mass value="0.16496568495572975"/>
     <inertia ixx="6.8e-05" iyy="6.8e-05" izz="7.3e-05" ixy="-2.4e-05" iyz="0.0" ixz="0.0"/>
@@ -566,5 +566,5 @@
 <link name="RB_DS51150_270_1_1">
   <inertial>
-    <origin xyz="-0.02303277025380847 0.023032770266688846 -0.006733285359181024" rpy="0 0 0"/>
+    <origin xyz="-0.023032770253802626 0.023032770266685404 -0.006733285359163047" rpy="0 0 0"/>
     <mass value="0.16496568495572975"/>
     <inertia ixx="6.8e-05" iyy="6.8e-05" izz="7.3e-05" ixy="2.4e-05" iyz="-0.0" ixz="0.0"/>
@@ -586,5 +586,5 @@
 <link name="LF_DS51150_270_1_1">
   <inertial>
-    <origin xyz="0.023032770253793314 -0.023032770266692065 -0.0067332853591978185" rpy="0 0 0"/>
+    <origin xyz="0.0230327702538011 -0.02303277026668407 -0.006733285359159725" rpy="0 0 0"/>
     <mass value="0.16496568495572975"/>
     <inertia ixx="6.8e-05" iyy="6.8e-05" izz="7.3e-05" ixy="2.4e-05" iyz="0.0" ixz="-0.0"/>
@@ -686,5 +686,5 @@
 <link name="RB_bearing_1_1">
   <inertial>
-    <origin xyz="-2.011289320369425e-07 2.0112892845647323e-07 -0.0020000000000233685" rpy="0 0 0"/>
+    <origin xyz="-2.011289298720076e-07 2.0112893012180777e-07 -0.0020000000000093623" rpy="0 0 0"/>
     <mass value="0.003999875766550524"/>
     <inertia ixx="0.0" iyy="0.0" izz="0.0" ixy="0.0" iyz="0.0" ixz="0.0"/>
@@ -706,7 +706,7 @@
 <link name="LF_bearing_1_1">
   <inertial>
-    <origin xyz="2.0112893234225382e-07 -2.0112894041912632e-07 -0.0020000000000358793" rpy="0 0 0"/>
+    <origin xyz="2.0112893564516732e-07 -2.0112893614476768e-07 -0.0020000000000144035" rpy="0 0 0"/>
     <mass value="0.003999875766550524"/>
-    <inertia ixx="0.0" iyy="0.0" izz="0.0" ixy="0.0" iyz="0.0" ixz="0.0"/>
+    <inertia ixx="0.0" iyy="0.0" izz="0.0" ixy="0.0" iyz="0.0" ixz="-0.0"/>
   </inertial>
   <visual>
@@ -1046,10 +1046,10 @@
 <link name="M_column_3_1">
   <inertial>
-    <origin xyz="-0.020000085460240125 0.013550502923226248 0.024026980815015697" rpy="0 0 0"/>
+    <origin xyz="0.019999914539759828 0.026450075088331488 -0.024026980815016585" rpy="0 0 0"/>
     <mass value="0.41107126565484164"/>
-    <inertia ixx="0.000227" iyy="0.000223" izz="0.000209" ixy="0.0" iyz="1.4e-05" ixz="0.0"/>
-  </inertial>
-  <visual>
-    <origin xyz="-0.020071 0.020071 -0.3391" rpy="0 0 0"/>
+    <inertia ixx="0.000227" iyy="0.000223" izz="0.000209" ixy="-0.0" iyz="1.4e-05" ixz="-0.0"/>
+  </inertial>
+  <visual>
+    <origin xyz="0.019929 0.020071 -0.3351" rpy="0 0 0"/>
     <geometry>
       <mesh filename="package://HEXAPEDAL_URDF_description/meshes/M_column_3_1.stl" scale="0.001 0.001 0.001"/>
@@ -1058,5 +1058,5 @@
   </visual>
   <collision>
-    <origin xyz="-0.020071 0.020071 -0.3391" rpy="0 0 0"/>
+    <origin xyz="0.019929 0.020071 -0.3351" rpy="0 0 0"/>
     <geometry>
       <mesh filename="package://HEXAPEDAL_URDF_description/meshes/M_column_3_1.stl" scale="0.001 0.001 0.001"/>
@@ -1064,21 +1064,21 @@
   </collision>
 </link>
-<link name="MID-360_4_2_1_1">
-  <inertial>
-    <origin xyz="0.018056496720877998 -0.021736152653647717 -0.010317011776493301" rpy="0 0 0"/>
-    <mass value="0.12034682690234494"/>
-    <inertia ixx="4.2e-05" iyy="5.2e-05" izz="7.3e-05" ixy="0.0" iyz="-1.8e-05" ixz="0.0"/>
-  </inertial>
-  <visual>
-    <origin xyz="0.017929 -0.004714 -0.393473" rpy="0 0 0"/>
-    <geometry>
-      <mesh filename="package://HEXAPEDAL_URDF_description/meshes/MID-360_4_2_1_1.stl" scale="0.001 0.001 0.001"/>
-    </geometry>
-    <material name="silver"/>
-  </visual>
-  <collision>
-    <origin xyz="0.017929 -0.004714 -0.393473" rpy="0 0 0"/>
-    <geometry>
-      <mesh filename="package://HEXAPEDAL_URDF_description/meshes/MID-360_4_2_1_1.stl" scale="0.001 0.001 0.001"/>
+<link name="livox_mid_360_1">
+  <inertial>
+    <origin xyz="-0.0180002892165137 -0.012662743628037466 -0.026067727094593318" rpy="0 0 0"/>
+    <mass value="1.055789101972525"/>
+    <inertia ixx="0.000443" iyy="0.000506" izz="0.000632" ixy="0.0" iyz="-0.000109" ixz="-0.0"/>
+  </inertial>
+  <visual>
+    <origin xyz="-0.018071 -0.036714 -0.304727" rpy="0 0 0"/>
+    <geometry>
+      <mesh filename="package://HEXAPEDAL_URDF_description/meshes/livox_mid_360_1.stl" scale="0.001 0.001 0.001"/>
+    </geometry>
+    <material name="silver"/>
+  </visual>
+  <collision>
+    <origin xyz="-0.018071 -0.036714 -0.304727" rpy="0 0 0"/>
+    <geometry>
+      <mesh filename="package://HEXAPEDAL_URDF_description/meshes/livox_mid_360_1.stl" scale="0.001 0.001 0.001"/>
     </geometry>
   </collision>
@@ -1086,5 +1086,5 @@
 <link name="LF_motor_horn_1_1">
   <inertial>
-    <origin xyz="2.0112882836986756e-07 -2.0112901788493787e-07 -0.0029620014636270384" rpy="0 0 0"/>
+    <origin xyz="2.0112883633571776e-07 -2.0112900966928748e-07 -0.0029620014635887496" rpy="0 0 0"/>
     <mass value="0.0019994583976964877"/>
     <inertia ixx="0.0" iyy="0.0" izz="0.0" ixy="0.0" iyz="-0.0" ixz="-0.0"/>
@@ -1126,5 +1126,5 @@
 <link name="LB_motor_horn_1_1">
   <inertial>
-    <origin xyz="2.011290100023544e-07 2.0112882784251163e-07 -0.0029620014636008683" rpy="0 0 0"/>
+    <origin xyz="2.0112900539492884e-07 2.0112883239442603e-07 -0.002962001463592448" rpy="0 0 0"/>
     <mass value="0.0019994583976964877"/>
     <inertia ixx="0.0" iyy="0.0" izz="0.0" ixy="-0.0" iyz="-0.0" ixz="0.0"/>
@@ -1186,5 +1186,5 @@
 <link name="RB_motor_horn_1_1">
   <inertial>
-    <origin xyz="-2.0112884444034584e-07 2.0112901552571394e-07 -0.0029620014636034253" rpy="0 0 0"/>
+    <origin xyz="-2.0112883974965357e-07 2.0112901288893426e-07 -0.0029620014635853113" rpy="0 0 0"/>
     <mass value="0.0019994583976964877"/>
     <inertia ixx="0.0" iyy="0.0" izz="0.0" ixy="0.0" iyz="0.0" ixz="0.0"/>
@@ -1226,5 +1226,5 @@
 <link name="RM_coxaR_1">
   <inertial>
-    <origin xyz="-0.03700000085533775 0.00042260385343186437 -0.034222602666993715" rpy="0 0 0"/>
+    <origin xyz="-0.037000000855337584 0.0004226038534422383 -0.03422260266699357" rpy="0 0 0"/>
     <mass value="0.09366200268610271"/>
     <inertia ixx="0.000108" iyy="0.000126" izz="0.000126" ixy="1e-06" iyz="-0.0" ixz="1e-06"/>
@@ -1246,5 +1246,5 @@
 <link name="RB_coxaR_1">
   <inertial>
-    <origin xyz="-0.025864326587127562 0.026461978688168936 -0.034222602667003915" rpy="0 0 0"/>
+    <origin xyz="-0.025864326587123065 0.02646197868816627 -0.034222602666985784" rpy="0 0 0"/>
     <mass value="0.09366200268610271"/>
     <inertia ixx="0.000118" iyy="0.000115" izz="0.000126" ixy="9e-06" iyz="-1e-06" ixz="1e-06"/>
@@ -1266,5 +1266,5 @@
 <link name="LF_coxaL_1">
   <inertial>
-    <origin xyz="0.026461977339766296 -0.0258643279355191 -0.03422260266704109" rpy="0 0 0"/>
+    <origin xyz="0.026461977339774206 -0.02586432793551094 -0.0342226026670027" rpy="0 0 0"/>
     <mass value="0.09366200268610271"/>
     <inertia ixx="0.000115" iyy="0.000118" izz="0.000126" ixy="9e-06" iyz="1e-06" ixz="-1e-06"/>
@@ -1306,5 +1306,5 @@
 <link name="LB_coxaL_1">
   <inertial>
-    <origin xyz="0.02586432793551041 0.026461977339764214 -0.0342226026670124" rpy="0 0 0"/>
+    <origin xyz="0.025864327935505804 0.026461977339768905 -0.03422260266700408" rpy="0 0 0"/>
     <mass value="0.09366200268610271"/>
     <inertia ixx="0.000118" iyy="0.000115" izz="0.000126" ixy="-9e-06" iyz="-1e-06" ixz="-1e-06"/>
@@ -1346,5 +1346,5 @@
 <link name="RM_motor_horn_2_1">
   <inertial>
-    <origin xyz="2.7755575615628914e-16 0.00386200146358686 -1.2329364841068194e-13" rpy="0 0 0"/>
+    <origin xyz="-1.2212453270876722e-15 0.003862001463596998 -1.2308238216877004e-13" rpy="0 0 0"/>
     <mass value="0.0019994583976964877"/>
     <inertia ixx="0.0" iyy="0.0" izz="0.0" ixy="0.0" iyz="0.0" ixz="-0.0"/>
@@ -1366,10 +1366,10 @@
 <link name="RB_motor_horn_2_1">
   <inertial>
-    <origin xyz="0.0027305352830171714 0.002730741156487887 -1.3337612854330877e-13" rpy="0 0 0"/>
+    <origin xyz="0.0027305352830218066 0.002730741156485167 -1.1531083698720926e-13" rpy="0 0 0"/>
     <mass value="0.0019994583976964877"/>
     <inertia ixx="0.0" iyy="0.0" izz="0.0" ixy="0.0" iyz="0.0" ixz="0.0"/>
   </inertial>
   <visual>
-    <origin xyz="0.206687 -0.158887 0.0" rpy="0 0 0"/>
+    <origin xyz="0.206687 -0.158887 -0.0" rpy="0 0 0"/>
     <geometry>
       <mesh filename="package://HEXAPEDAL_URDF_description/meshes/RB_motor_horn_2_1.stl" scale="0.001 0.001 0.001"/>
@@ -1378,5 +1378,5 @@
   </visual>
   <collision>
-    <origin xyz="0.206687 -0.158887 0.0" rpy="0 0 0"/>
+    <origin xyz="0.206687 -0.158887 -0.0" rpy="0 0 0"/>
     <geometry>
       <mesh filename="package://HEXAPEDAL_URDF_description/meshes/RB_motor_horn_2_1.stl" scale="0.001 0.001 0.001"/>
@@ -1386,10 +1386,10 @@
 <link name="LF_motor_horn_2_1">
   <inertial>
-    <origin xyz="0.002730741156475508 0.002730535283013563 8.548115031890303e-14" rpy="0 0 0"/>
+    <origin xyz="0.0027307411564834183 0.0027305352830214458 1.2307251773562983e-13" rpy="0 0 0"/>
     <mass value="0.0019994583976964877"/>
     <inertia ixx="0.0" iyy="0.0" izz="0.0" ixy="0.0" iyz="-0.0" ixz="-0.0"/>
   </inertial>
   <visual>
-    <origin xyz="-0.158887 0.206687 0.0" rpy="0 0 0"/>
+    <origin xyz="-0.158887 0.206687 -0.0" rpy="0 0 0"/>
     <geometry>
       <mesh filename="package://HEXAPEDAL_URDF_description/meshes/LF_motor_horn_2_1.stl" scale="0.001 0.001 0.001"/>
@@ -1398,5 +1398,5 @@
   </visual>
   <collision>
-    <origin xyz="-0.158887 0.206687 0.0" rpy="0 0 0"/>
+    <origin xyz="-0.158887 0.206687 -0.0" rpy="0 0 0"/>
     <geometry>
       <mesh filename="package://HEXAPEDAL_URDF_description/meshes/LF_motor_horn_2_1.stl" scale="0.001 0.001 0.001"/>
@@ -1426,5 +1426,5 @@
 <link name="LB_motor_horn_2_1">
   <inertial>
-    <origin xyz="-0.0027305352830239438 0.0027307411564732598 1.1333888079242351e-13" rpy="0 0 0"/>
+    <origin xyz="-0.0027305352830285234 0.002730741156477867 1.216963209818856e-13" rpy="0 0 0"/>
     <mass value="0.0019994583976964877"/>
     <inertia ixx="0.0" iyy="0.0" izz="0.0" ixy="-0.0" iyz="-0.0" ixz="0.0"/>
@@ -1446,10 +1446,10 @@
 <link name="LF_DS51150_270_2_1">
   <inertial>
-    <origin xyz="0.03560985654621199 0.008136788935386469 9.072852876170052e-12" rpy="0 0 0"/>
+    <origin xyz="0.03560985654621959 0.008136788935394268 9.110513602833456e-12" rpy="0 0 0"/>
     <mass value="0.16496568495572975"/>
     <inertia ixx="5.8e-05" iyy="5.9e-05" izz="9.3e-05" ixy="1.5e-05" iyz="0.0" ixz="0.0"/>
   </inertial>
   <visual>
-    <origin xyz="-0.159523 0.206051 0.0" rpy="0 0 0"/>
+    <origin xyz="-0.159523 0.206051 -0.0" rpy="0 0 0"/>
     <geometry>
       <mesh filename="package://HEXAPEDAL_URDF_description/meshes/LF_DS51150_270_2_1.stl" scale="0.001 0.001 0.001"/>
@@ -1458,5 +1458,5 @@
   </visual>
   <collision>
-    <origin xyz="-0.159523 0.206051 0.0" rpy="0 0 0"/>
+    <origin xyz="-0.159523 0.206051 -0.0" rpy="0 0 0"/>
     <geometry>
       <mesh filename="package://HEXAPEDAL_URDF_description/meshes/LF_DS51150_270_2_1.stl" scale="0.001 0.001 0.001"/>
@@ -1466,5 +1466,5 @@
 <link name="LM_DS51150_270_2_1">
   <inertial>
-    <origin xyz="0.019426246833090577 0.03093328535916428 9.10862149369396e-12" rpy="0 0 0"/>
+    <origin xyz="0.01942624683309052 0.03093328535916428 9.108625902271619e-12" rpy="0 0 0"/>
     <mass value="0.16496568495572975"/>
     <inertia ixx="4.4e-05" iyy="7.3e-05" izz="9.3e-05" ixy="-0.0" iyz="0.0" ixz="-0.0"/>
@@ -1486,5 +1486,5 @@
 <link name="LB_DS51150_270_2_1">
   <inertial>
-    <origin xyz="-0.008136788935395461 0.03560985654620624 9.100279146254787e-12" rpy="0 0 0"/>
+    <origin xyz="-0.008136788935400124 0.03560985654621082 9.108673217267947e-12" rpy="0 0 0"/>
     <mass value="0.16496568495572975"/>
     <inertia ixx="5.9e-05" iyy="5.8e-05" izz="9.3e-05" ixy="-1.5e-05" iyz="0.0" ixz="-0.0"/>
@@ -1526,5 +1526,5 @@
 <link name="RM_DS51150_270_2_1">
   <inertial>
-    <origin xyz="-0.019426246833087912 0.03093328535915816 -9.10996944823753e-12" rpy="0 0 0"/>
+    <origin xyz="-0.01942624683308497 0.03093328535917127 -9.111592340665953e-12" rpy="0 0 0"/>
     <mass value="0.16496568495572975"/>
     <inertia ixx="4.4e-05" iyy="7.3e-05" izz="9.3e-05" ixy="0.0" iyz="-0.0" ixz="-0.0"/>
@@ -1546,10 +1546,10 @@
 <link name="RB_DS51150_270_2_1">
   <inertial>
-    <origin xyz="0.0081367889353893 0.035609856546221175 -9.120399476032414e-12" rpy="0 0 0"/>
+    <origin xyz="0.00813678893539413 0.03560985654621854 -9.102308010916462e-12" rpy="0 0 0"/>
     <mass value="0.16496568495572975"/>
     <inertia ixx="5.9e-05" iyy="5.8e-05" izz="9.3e-05" ixy="1.5e-05" iyz="-0.0" ixz="-0.0"/>
   </inertial>
   <visual>
-    <origin xyz="0.206051 -0.159523 0.0" rpy="0 0 0"/>
+    <origin xyz="0.206051 -0.159523 -0.0" rpy="0 0 0"/>
     <geometry>
       <mesh filename="package://HEXAPEDAL_URDF_description/meshes/RB_DS51150_270_2_1.stl" scale="0.001 0.001 0.001"/>
@@ -1558,5 +1558,5 @@
   </visual>
   <collision>
-    <origin xyz="0.206051 -0.159523 0.0" rpy="0 0 0"/>
+    <origin xyz="0.206051 -0.159523 -0.0" rpy="0 0 0"/>
     <geometry>
       <mesh filename="package://HEXAPEDAL_URDF_description/meshes/RB_DS51150_270_2_1.stl" scale="0.001 0.001 0.001"/>
@@ -1564,7 +1564,27 @@
   </collision>
 </link>
+<link name="mid-360-fov-asm_ver.ksh_MID-360_4_1_1_1">
+  <inertial>
+    <origin xyz="-2.784486891456114e-07 0.005174945755449259 -0.008963272176272019" rpy="0 0 0"/>
+    <mass value="0.2760142598595122"/>
+    <inertia ixx="4.7e-05" iyy="5.2e-05" izz="6.2e-05" ixy="-0.0" iyz="-9e-06" ixz="-0.0"/>
+  </inertial>
+  <visual>
+    <origin xyz="-7.1e-05 -0.033453 -0.262375" rpy="0 0 0"/>
+    <geometry>
+      <mesh filename="package://HEXAPEDAL_URDF_description/meshes/mid-360-fov-asm_ver.ksh_MID-360_4_1_1_1.stl" scale="0.001 0.001 0.001"/>
+    </geometry>
+    <material name="silver"/>
+  </visual>
+  <collision>
+    <origin xyz="-7.1e-05 -0.033453 -0.262375" rpy="0 0 0"/>
+    <geometry>
+      <mesh filename="package://HEXAPEDAL_URDF_description/meshes/mid-360-fov-asm_ver.ksh_MID-360_4_1_1_1.stl" scale="0.001 0.001 0.001"/>
+    </geometry>
+  </collision>
+</link>
 <link name="RF_link1_right_1">
   <inertial>
-    <origin xyz="-0.022677021050098972 -0.03745516077457217 -0.015609126867096599" rpy="0 0 0"/>
+    <origin xyz="-0.022677020519566077 -0.037455160000820775 -0.015609126867096363" rpy="0 0 0"/>
     <mass value="0.05250233789665554"/>
     <inertia ixx="6.3e-05" iyy="6.3e-05" izz="0.000106" ixy="-4.5e-05" iyz="-1e-06" ixz="1e-06"/>
@@ -1586,5 +1606,5 @@
 <link name="RF_DS51150_270_3_1">
   <inertial>
-    <origin xyz="0.017106763797174407 -0.017211590721209924 -0.01499999999089773" rpy="0 0 0"/>
+    <origin xyz="0.017106763843891093 -0.017211590398439225 -0.014999999990897343" rpy="0 0 0"/>
     <mass value="0.16496568495572975"/>
     <inertia ixx="5.9e-05" iyy="5.8e-05" izz="9.3e-05" ixy="-1.5e-05" iyz="0.0" ixz="-0.0"/>
@@ -1606,5 +1626,5 @@
 <link name="RF_bearing_2_1">
   <inertial>
-    <origin xyz="-0.0014145445240567045 0.0014139128534798595 -7.793169765454425e-15" rpy="0 0 0"/>
+    <origin xyz="-0.0014145438679431521 0.001413913558223956 -7.574574939285309e-15" rpy="0 0 0"/>
     <mass value="0.003999875766550524"/>
     <inertia ixx="0.0" iyy="0.0" izz="0.0" ixy="-0.0" iyz="0.0" ixz="0.0"/>
@@ -1626,5 +1646,5 @@
 <link name="RF_bearing_3_1">
   <inertial>
-    <origin xyz="-0.00141457383079302 0.0014138835467424338 -6.671790675630351e-15" rpy="0 0 0"/>
+    <origin xyz="-0.001414573372445882 0.0014138844492528058 -6.518651033802115e-15" rpy="0 0 0"/>
     <mass value="0.003999875766550524"/>
     <inertia ixx="0.0" iyy="0.0" izz="0.0" ixy="-0.0" iyz="0.0" ixz="-0.0"/>
@@ -1646,5 +1666,5 @@
 <link name="RM_link1_right_1">
   <inertial>
-    <origin xyz="-0.04251961166602958 -0.010449696254225434 -0.01560912686708989" rpy="0 0 0"/>
+    <origin xyz="-0.04251961074375893 -0.010449696082221856 -0.015609126867088947" rpy="0 0 0"/>
     <mass value="0.05250233789665554"/>
     <inertia ixx="1.8e-05" iyy="0.000108" izz="0.000106" ixy="0.0" iyz="-1e-06" ixz="0.0"/>
@@ -1666,5 +1686,5 @@
 <link name="RM_DS51150_270_3_1">
   <inertial>
-    <origin xyz="-7.375391196973169e-05 -0.02426671464084055 -0.014999999990891074" rpy="0 0 0"/>
+    <origin xyz="-7.375365070272366e-05 -0.02426671444562294 -0.014999999990891844" rpy="0 0 0"/>
     <mass value="0.16496568495572975"/>
     <inertia ixx="4.4e-05" iyy="7.3e-05" izz="9.3e-05" ixy="-0.0" iyz="0.0" ixz="-0.0"/>
@@ -1686,7 +1706,7 @@
 <link name="RM_bearing_2_1">
   <inertial>
-    <origin xyz="9.387737254229478e-10 0.0019999999999936666 -9.936434388075706e-16" rpy="0 0 0"/>
+    <origin xyz="1.9010492624538244e-09 0.0020000000343989334 -1.0595268767677703e-15" rpy="0 0 0"/>
     <mass value="0.003999875766550524"/>
-    <inertia ixx="0.0" iyy="0.0" izz="0.0" ixy="0.0" iyz="0.0" ixz="-0.0"/>
+    <inertia ixx="0.0" iyy="0.0" izz="0.0" ixy="0.0" iyz="-0.0" ixz="-0.0"/>
   </inertial>
   <visual>
@@ -1706,247 +1726,247 @@
 <link name="RM_bearing_3_1">
   <inertial>
-    <origin xyz="-1.89244730997018e-09 0.0019999999999949607 3.74119312038047e-17" rpy="0 0 0"/>
+    <origin xyz="-9.301727721400255e-10 0.0020000003140845067 -2.076281183175288e-15" rpy="0 0 0"/>
+    <mass value="0.003999875766550524"/>
+    <inertia ixx="0.0" iyy="0.0" izz="0.0" ixy="0.0" iyz="-0.0" ixz="-0.0"/>
+  </inertial>
+  <visual>
+    <origin xyz="0.3825 -0.0273 -0.0" rpy="0 0 0"/>
+    <geometry>
+      <mesh filename="package://HEXAPEDAL_URDF_description/meshes/RM_bearing_3_1.stl" scale="0.001 0.001 0.001"/>
+    </geometry>
+    <material name="silver"/>
+  </visual>
+  <collision>
+    <origin xyz="0.3825 -0.0273 -0.0" rpy="0 0 0"/>
+    <geometry>
+      <mesh filename="package://HEXAPEDAL_URDF_description/meshes/RM_bearing_3_1.stl" scale="0.001 0.001 0.001"/>
+    </geometry>
+  </collision>
+</link>
+<link name="RB_link1_right_1">
+  <inertial>
+    <origin xyz="-0.03745516000082588 0.022677020519567354 -0.015609126867082355" rpy="0 0 0"/>
+    <mass value="0.05250233789665554"/>
+    <inertia ixx="6.3e-05" iyy="6.3e-05" izz="0.000106" ixy="4.5e-05" iyz="-1e-06" ixz="-1e-06"/>
+  </inertial>
+  <visual>
+    <origin xyz="0.180807 -0.212344 -0.015" rpy="0 0 0"/>
+    <geometry>
+      <mesh filename="package://HEXAPEDAL_URDF_description/meshes/RB_link1_right_1.stl" scale="0.001 0.001 0.001"/>
+    </geometry>
+    <material name="silver"/>
+  </visual>
+  <collision>
+    <origin xyz="0.180807 -0.212344 -0.015" rpy="0 0 0"/>
+    <geometry>
+      <mesh filename="package://HEXAPEDAL_URDF_description/meshes/RB_link1_right_1.stl" scale="0.001 0.001 0.001"/>
+    </geometry>
+  </collision>
+</link>
+<link name="RB_DS51150_270_3_1">
+  <inertial>
+    <origin xyz="-0.017211590398443666 -0.017106763843889927 -0.014999999990883821" rpy="0 0 0"/>
+    <mass value="0.16496568495572975"/>
+    <inertia ixx="5.8e-05" iyy="5.9e-05" izz="9.3e-05" ixy="1.5e-05" iyz="0.0" ixz="0.0"/>
+  </inertial>
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
Commit message: fix(urdf): align Livox frame with Fusion axes

File: HW/urdf/urdf/HEXAPEDAL_URDF.xacro (robot description, xacro)
@@ -1066,10 +1066,10 @@
 <link name="livox_mid_360_1">
   <inertial>
-    <origin xyz="-0.0180002892165137 -0.012662743628037466 -0.026067727094593318" rpy="0 0 0"/>
+    <origin xyz="-0.024 0.018 -0.016243934732367332" rpy="0 0 0"/>
     <mass value="1.055789101972525"/>
-    <inertia ixx="0.000443" iyy="0.000506" izz="0.000632" ixy="0.0" iyz="-0.000109" ixz="-0.0"/>
-  </inertial>
-  <visual>
-    <origin xyz="-0.018071 -0.036714 -0.304727" rpy="0 0 0"/>
+    <inertia ixx="0.00044310323098749614" iyy="0.000443" izz="0.0006948967690125037" ixy="0.0" iyz="0.0" ixz="5.9600438419613695e-8"/>
+  </inertial>
+  <visual>
+    <origin xyz="-0.18415863546375527 0.01807071078348564 -0.24554431588256895" rpy="-0.5235987755982988 0 -1.5707963267948966"/>
     <geometry>
       <mesh filename="package://HEXAPEDAL_URDF_description/meshes/livox_mid_360_1.stl" scale="0.001 0.001 0.001"/>
@@ -1078,5 +1078,5 @@
   </visual>
   <collision>
-    <origin xyz="-0.018071 -0.036714 -0.304727" rpy="0 0 0"/>
+    <origin xyz="-0.18415863546375527 0.01807071078348564 -0.24554431588256895" rpy="-0.5235987755982988 0 -1.5707963267948966"/>
     <geometry>
       <mesh filename="package://HEXAPEDAL_URDF_description/meshes/livox_mid_360_1.stl" scale="0.001 0.001 0.001"/>
@@ -2925,5 +2925,6 @@
 </joint>
 <joint name="강체 202" type="fixed">
-  <origin xyz="0.038 0.056785 -0.030373" rpy="0 0 0"/>
+  <!-- Fusion joint geometryOne: red X, green Y, blue Z. -->
+  <origin xyz="0.03799971078348564 0.0567848986966054 -0.03037306695894683" rpy="0 -0.5235987755982988 1.5707963267948966"/>
   <parent link="M_column_3_1"/>
   <child link="livox_mid_360_1"/>
@@ -3074,5 +3075,6 @@
 </joint>
 <joint name="강체 201" type="fixed">
-  <origin xyz="-0.018 -0.003261 -0.042352" rpy="0 0 0"/>
+  <!-- Counter-transform keeps the FOV mesh at its original world pose. -->
+  <origin xyz="-0.024 0.018 -0.035047" rpy="-0.5235987755982988 0 -1.5707963267948966"/>
   <parent link="livox_mid_360_1"/>
   <child link="mid-360-fov-asm_ver.ksh_MID-360_4_1_1_1"/>
