Commit message: feat(urdf): update model and Livox frame

File: HW/urdf/urdf/HEXAPEDAL_URDF.xacro (robot description, xacro)
@@ -1046,7 +1046,7 @@
 <link name="M_column_3_1">
   <inertial>
-    <origin xyz="0.019999914539759828 0.026450075088331488 -0.024026980815016585" rpy="0 0 0"/>
-    <mass value="0.41107126565484164"/>
-    <inertia ixx="0.000227" iyy="0.000223" izz="0.000209" ixy="-0.0" iyz="1.4e-05" ixz="-0.0"/>
+    <origin xyz="0.0199997107796305 0.027043537648551216 -0.033112260347502476" rpy="0 0 0"/>
+    <mass value="0.48244290405365176"/>
+    <inertia ixx="0.000378" iyy="0.000363" izz="0.000251" ixy="-0.0" iyz="5.6e-05" ixz="0.0"/>
   </inertial>
   <visual>
@@ -1061,24 +1061,4 @@
     <geometry>
       <mesh filename="package://HEXAPEDAL_URDF_description/meshes/M_column_3_1.stl" scale="0.001 0.001 0.001"/>
-    </geometry>
-  </collision>
-</link>
-<link name="livox_mid_360_1">
-  <inertial>
-    <origin xyz="-0.024 0.018 -0.016243934732367332" rpy="0 0 0"/>
-    <mass value="1.055789101972525"/>
-    <inertia ixx="0.00044310323098749614" iyy="0.000443" izz="0.0006948967690125037" ixy="0.0" iyz="0.0" ixz="5.9600438419613695e-8"/>
-  </inertial>
-  <visual>
-    <origin xyz="-0.18415863546375527 0.01807071078348564 -0.24554431588256895" rpy="-0.5235987755982988 0 -1.5707963267948966"/>
-    <geometry>
-      <mesh filename="package://HEXAPEDAL_URDF_description/meshes/livox_mid_360_1.stl" scale="0.001 0.001 0.001"/>
-    </geometry>
-    <material name="silver"/>
-  </visual>
-  <collision>
-    <origin xyz="-0.18415863546375527 0.01807071078348564 -0.24554431588256895" rpy="-0.5235987755982988 0 -1.5707963267948966"/>
-    <geometry>
-      <mesh filename="package://HEXAPEDAL_URDF_description/meshes/livox_mid_360_1.stl" scale="0.001 0.001 0.001"/>
     </geometry>
   </collision>
@@ -1564,21 +1544,21 @@
   </collision>
 </link>
-<link name="mid-360-fov-asm_ver.ksh_MID-360_4_1_1_1">
-  <inertial>
-    <origin xyz="-2.784486891456114e-07 0.005174945755449259 -0.008963272176272019" rpy="0 0 0"/>
-    <mass value="0.2760142598595122"/>
-    <inertia ixx="4.7e-05" iyy="5.2e-05" izz="6.2e-05" ixy="-0.0" iyz="-9e-06" ixz="-0.0"/>
-  </inertial>
-  <visual>
-    <origin xyz="-7.1e-05 -0.033453 -0.262375" rpy="0 0 0"/>
-    <geometry>
-      <mesh filename="package://HEXAPEDAL_URDF_description/meshes/mid-360-fov-asm_ver.ksh_MID-360_4_1_1_1.stl" scale="0.001 0.001 0.001"/>
-    </geometry>
-    <material name="silver"/>
-  </visual>
-  <collision>
-    <origin xyz="-7.1e-05 -0.033453 -0.262375" rpy="0 0 0"/>
-    <geometry>
-      <mesh filename="package://HEXAPEDAL_URDF_description/meshes/mid-360-fov-asm_ver.ksh_MID-360_4_1_1_1.stl" scale="0.001 0.001 0.001"/>
+<link name="livox_mid_360_1">
+  <inertial>
+    <origin xyz="0.02399969341720557 0.01799971078348498 0.016243790042632766" rpy="3.141592653589793 0 1.5707963267948966"/>
+    <mass value="1.055789101972525"/>
+    <inertia ixx="0.000444" iyy="0.000443" izz="0.000694" ixy="-0.0" iyz="-0.0" ixz="-0.0"/>
+  </inertial>
+  <visual>
+    <origin xyz="0.011962306582794429 0.01792928921651436 0.2746291446897346" rpy="3.141592653589793 0 1.5707963267948966"/>
+    <geometry>
+      <mesh filename="package://HEXAPEDAL_URDF_description/meshes/livox_mid_360_1.stl" scale="0.001 0.001 0.001"/>
+    </geometry>
+    <material name="silver"/>
+  </visual>
+  <collision>
+    <origin xyz="0.011962306582794429 0.01792928921651436 0.2746291446897346" rpy="3.141592653589793 0 1.5707963267948966"/>
+    <geometry>
+      <mesh filename="package://HEXAPEDAL_URDF_description/meshes/livox_mid_360_1.stl" scale="0.001 0.001 0.001"/>
     </geometry>
   </collision>
@@ -2064,4 +2044,24 @@
   </collision>
 </link>
+<link name="mid-360-fov-asm_ver.ksh_MID-360_4_1_1_1">
+  <inertial>
+    <origin xyz="-2.999843395723136e-07 -3.1735112955566525e-07 -0.010350150158302679" rpy="0 0 0"/>
+    <mass value="0.2760142598595122"/>
+    <inertia ixx="4.7e-05" iyy="4.7e-05" izz="6.7e-05" ixy="-0.0" iyz="0.0" ixz="0.0"/>
+  </inertial>
+  <visual>
+    <origin xyz="-7.1e-05 -0.012038 -0.239582" rpy="0 0 0"/>
+    <geometry>
+      <mesh filename="package://HEXAPEDAL_URDF_description/meshes/mid-360-fov-asm_ver.ksh_MID-360_4_1_1_1.stl" scale="0.001 0.001 0.001"/>
+    </geometry>
+    <material name="silver"/>
+  </visual>
+  <collision>
+    <origin xyz="-7.1e-05 -0.012038 -0.239582" rpy="0 0 0"/>
+    <geometry>
+      <mesh filename="package://HEXAPEDAL_URDF_description/meshes/mid-360-fov-asm_ver.ksh_MID-360_4_1_1_1.stl" scale="0.001 0.001 0.001"/>
+    </geometry>
+  </collision>
+</link>
 <link name="LF_motor_horn_3_1">
   <inertial>
@@ -2306,10 +2306,10 @@
 <link name="LF_foot_1_1">
   <inertial>
-    <origin xyz="-0.019873692600057113 0.01987360562351681 0.003538514539441144" rpy="0 0 0"/>
-    <mass value="0.17136403212360193"/>
-    <inertia ixx="3.5e-05" iyy="3.5e-05" izz="5.8e-05" ixy="1.1e-05" iyz="-0.0" ixz="0.0"/>
-  </inertial>
-  <visual>
-    <origin xyz="-0.422058 0.421775 0.015171" rpy="0 0 0"/>
+    <origin xyz="-0.006116804265747233 -0.009539635368250199 -0.003649088182073809" rpy="0 0 0"/>
+    <mass value="0.1874472710453902"/>
+    <inertia ixx="4.3e-05" iyy="4.3e-05" izz="7.2e-05" ixy="1.1e-05" iyz="-1e-06" ixz="-0.0"/>
+  </inertial>
+  <visual>
+    <origin xyz="-0.408461 0.393402 -0.015489" rpy="0 0 0"/>
     <geometry>
       <mesh filename="package://HEXAPEDAL_URDF_description/meshes/LF_foot_1_1.stl" scale="0.001 0.001 0.001"/>
@@ -2318,5 +2318,5 @@
   </visual>
   <collision>
-    <origin xyz="-0.422058 0.421775 0.015171" rpy="0 0 0"/>
+    <origin xyz="-0.408461 0.393402 -0.015489" rpy="0 0 0"/>
     <geometry>
       <mesh filename="package://HEXAPEDAL_URDF_description/meshes/LF_foot_1_1.stl" scale="0.001 0.001 0.001"/>
@@ -2326,10 +2326,10 @@
 <link name="LM_foot_1_1">
   <inertial>
-    <origin xyz="-0.028105547618765825 4.971735864794653e-08 0.0035385145394440827" rpy="0 0 0"/>
-    <mass value="0.17136403212360193"/>
-    <inertia ixx="2.4e-05" iyy="4.6e-05" izz="5.8e-05" ixy="-0.0" iyz="-0.0" ixz="0.0"/>
-  </inertial>
-  <visual>
-    <origin xyz="-0.59668 -0.0002 0.015171" rpy="0 0 0"/>
+    <origin xyz="0.0024210719660052726 0.009825546383462896 -0.003649088182036391" rpy="0 0 0"/>
+    <mass value="0.1874472710453902"/>
+    <inertia ixx="3.2e-05" iyy="5.3e-05" izz="7.2e-05" ixy="-0.0" iyz="-1e-06" ixz="0.0"/>
+  </inertial>
+  <visual>
+    <origin xyz="-0.567002 0.010248 -0.015489" rpy="0 0 0"/>
     <geometry>
       <mesh filename="package://HEXAPEDAL_URDF_description/meshes/LM_foot_1_1.stl" scale="0.001 0.001 0.001"/>
@@ -2338,5 +2338,5 @@
   </visual>
   <collision>
-    <origin xyz="-0.59668 -0.0002 0.015171" rpy="0 0 0"/>
+    <origin xyz="-0.567002 0.010248 -0.015489" rpy="0 0 0"/>
     <geometry>
       <mesh filename="package://HEXAPEDAL_URDF_description/meshes/LM_foot_1_1.stl" scale="0.001 0.001 0.001"/>
@@ -2346,10 +2346,10 @@
 <link name="LB_foot_1_1">
   <inertial>
-    <origin xyz="-0.019873605623526525 -0.019873692600071102 0.0035385145394379557" rpy="0 0 0"/>
-    <mass value="0.17136403212360193"/>
-    <inertia ixx="3.5e-05" iyy="3.5e-05" izz="5.8e-05" ixy="-1.1e-05" iyz="0.0" ixz="0.0"/>
-  </inertial>
-  <visual>
-    <origin xyz="-0.421775 -0.422058 0.015171" rpy="0 0 0"/>
+    <origin xyz="-0.005236364631764634 0.008659195734242175 -0.003649088182048536" rpy="0 0 0"/>
+    <mass value="0.1874472710453902"/>
+    <inertia ixx="4.3e-05" iyy="4.3e-05" izz="7.2e-05" ixy="-1.1e-05" iyz="-0.0" ixz="1e-06"/>
+  </inertial>
+  <visual>
+    <origin xyz="-0.408178 -0.393685 -0.015489" rpy="0 0 0"/>
     <geometry>
       <mesh filename="package://HEXAPEDAL_URDF_description/meshes/LB_foot_1_1.stl" scale="0.001 0.001 0.001"/>
@@ -2358,5 +2358,5 @@
   </visual>
   <collision>
-    <origin xyz="-0.421775 -0.422058 0.015171" rpy="0 0 0"/>
+    <origin xyz="-0.408178 -0.393685 -0.015489" rpy="0 0 0"/>
     <geometry>
       <mesh filename="package://HEXAPEDAL_URDF_description/meshes/LB_foot_1_1.stl" scale="0.001 0.001 0.001"/>
@@ -2366,10 +2366,10 @@
 <link name="RF_foot_1_1">
   <inertial>
-    <origin xyz="0.019873535171129997 0.019874070171167657 0.0035385442328290436" rpy="0 0 0"/>
-    <mass value="0.17136403212360193"/>
-    <inertia ixx="3.5e-05" iyy="3.5e-05" izz="5.8e-05" ixy="-1.1e-05" iyz="-0.0" ixz="-0.0"/>
-  </inertial>
-  <visual>
-    <origin xyz="0.422059 0.421775 0.015171" rpy="0 0 0"/>
+    <origin xyz="-0.008659195734254665 0.005236364631767243 0.00364908818203203" rpy="0 0 0"/>
+    <mass value="0.1874472710453902"/>
+    <inertia ixx="4.3e-05" iyy="4.3e-05" izz="7.2e-05" ixy="-1.1e-05" iyz="1e-06" ixz="-0.0"/>
+  </inertial>
+  <visual>
+    <origin xyz="0.393685 0.408178 0.015489" rpy="0 0 0"/>
     <geometry>
       <mesh filename="package://HEXAPEDAL_URDF_description/meshes/RF_foot_1_1.stl" scale="0.001 0.001 0.001"/>
@@ -2378,5 +2378,5 @@
   </visual>
   <collision>
-    <origin xyz="0.422059 0.421775 0.015171" rpy="0 0 0"/>
+    <origin xyz="0.393685 0.408178 0.015489" rpy="0 0 0"/>
     <geometry>
       <mesh filename="package://HEXAPEDAL_URDF_description/meshes/RF_foot_1_1.stl" scale="0.001 0.001 0.001"/>
@@ -2386,10 +2386,10 @@
 <link name="RM_foot_1_1">
   <inertial>
-    <origin xyz="0.028106057677708907 1.966280456167568e-07 0.003538544232830499" rpy="0 0 0"/>
-    <mass value="0.17136403212360193"/>
-    <inertia ixx="2.4e-05" iyy="4.6e-05" izz="5.8e-05" ixy="-0.0" iyz="0.0" ixz="-0.0"/>
-  </inertial>
-  <visual>
-    <origin xyz="0.596681 -0.000201 0.015171" rpy="0 0 0"/>
+    <origin xyz="-0.0024210719660007207 0.009825546383458925 0.00364908818203934" rpy="0 0 0"/>
+    <mass value="0.1874472710453902"/>
+    <inertia ixx="3.2e-05" iyy="5.3e-05" izz="7.2e-05" ixy="0.0" iyz="1e-06" ixz="0.0"/>
+  </inertial>
+  <visual>
+    <origin xyz="0.567002 0.010248 0.015489" rpy="0 0 0"/>
     <geometry>
       <mesh filename="package://HEXAPEDAL_URDF_description/meshes/RM_foot_1_1.stl" scale="0.001 0.001 0.001"/>
@@ -2398,5 +2398,5 @@
   </visual>
   <collision>
-    <origin xyz="0.596681 -0.000201 0.015171" rpy="0 0 0"/>
+    <origin xyz="0.567002 0.010248 0.015489" rpy="0 0 0"/>
     <geometry>
       <mesh filename="package://HEXAPEDAL_URDF_description/meshes/RM_foot_1_1.stl" scale="0.001 0.001 0.001"/>
@@ -2406,10 +2406,10 @@
 <link name="RB_foot_1_1">
   <inertial>
-    <origin xyz="0.019874070171163605 -0.019873535171128887 0.0035385442328431157" rpy="0 0 0"/>
-    <mass value="0.17136403212360193"/>
-    <inertia ixx="3.5e-05" iyy="3.5e-05" izz="5.8e-05" ixy="1.1e-05" iyz="0.0" ixz="-0.0"/>
-  </inertial>
-  <visual>
-    <origin xyz="0.421775 -0.422059 0.015171" rpy="0 0 0"/>
+    <origin xyz="-0.009539635368240762 -0.006116804265741627 0.0036490881820279257" rpy="0 0 0"/>
+    <mass value="0.1874472710453902"/>
+    <inertia ixx="4.3e-05" iyy="4.3e-05" izz="7.2e-05" ixy="1.1e-05" iyz="0.0" ixz="1e-06"/>
+  </inertial>
+  <visual>
+    <origin xyz="0.393402 -0.408461 0.015489" rpy="0 0 0"/>
     <geometry>
       <mesh filename="package://HEXAPEDAL_URDF_description/meshes/RB_foot_1_1.stl" scale="0.001 0.001 0.001"/>
@@ -2418,5 +2418,5 @@
   </visual>
   <collision>
-    <origin xyz="0.421775 -0.422059 0.015171" rpy="0 0 0"/>
+    <origin xyz="0.393402 -0.408461 0.015489" rpy="0 0 0"/>
     <geometry>
       <mesh filename="package://HEXAPEDAL_URDF_description/meshes/RB_foot_1_1.stl" scale="0.001 0.001 0.001"/>
@@ -2426,10 +2426,10 @@
 <link name="LF_foot_2_1">
   <inertial>
-    <origin xyz="0.001935672605184624 -0.001935898564140115 0.011535157888890112" rpy="0 0 0"/>
-    <mass value="0.1674566879251433"/>
-    <inertia ixx="3.5e-05" iyy="3.5e-05" izz="5.8e-05" ixy="1.1e-05" iyz="0.0" ixz="-0.0"/>
-  </inertial>
-  <visual>
-    <origin xyz="-0.400284 0.400001 -0.0" rpy="0 0 0"/>
+    <origin xyz="0.008808231577610404 0.005426310424457348 0.003691103892641016" rpy="0 0 0"/>
+    <mass value="0.1824085742487717"/>
+    <inertia ixx="4.2e-05" iyy="4.2e-05" izz="7e-05" ixy="1.1e-05" iyz="1e-06" ixz="0.0"/>
+  </inertial>
+  <visual>
+    <origin xyz="-0.393685 0.408178 0.015489" rpy="0 0 0"/>
     <geometry>
       <mesh filename="package://HEXAPEDAL_URDF_description/meshes/LF_foot_2_1.stl" scale="0.001 0.001 0.001"/>
@@ -2438,5 +2438,5 @@
   </visual>
   <collision>
-    <origin xyz="-0.400284 0.400001 -0.0" rpy="0 0 0"/>
+    <origin xyz="-0.393685 0.408178 0.015489" rpy="0 0 0"/>
     <geometry>
       <mesh filename="package://HEXAPEDAL_URDF_description/meshes/LF_foot_2_1.stl" scale="0.001 0.001 0.001"/>
@@ -2446,10 +2446,10 @@
 <link name="LM_foot_2_1">
   <inertial>
-    <origin xyz="0.0027375646095293416 -4.8558061535971175e-08 0.0115351578889062" rpy="0 0 0"/>
-    <mass value="0.1674566879251433"/>
-    <inertia ixx="2.4e-05" iyy="4.5e-05" izz="5.8e-05" ixy="0.0" iyz="-0.0" ixz="-0.0"/>
-  </inertial>
-  <visual>
-    <origin xyz="-0.565887 -0.0002 -0.0" rpy="0 0 0"/>
+    <origin xyz="0.002392144263401952 -0.010830757402977929 0.003691103892678507" rpy="0 0 0"/>
+    <mass value="0.1824085742487717"/>
+    <inertia ixx="3.1e-05" iyy="5.2e-05" izz="7e-05" ixy="-0.0" iyz="1e-06" ixz="-0.0"/>
+  </inertial>
+  <visual>
+    <origin xyz="-0.567002 -0.010648 0.015489" rpy="0 0 0"/>
     <geometry>
       <mesh filename="package://HEXAPEDAL_URDF_description/meshes/LM_foot_2_1.stl" scale="0.001 0.001 0.001"/>
@@ -2458,5 +2458,5 @@
   </visual>
   <collision>
-    <origin xyz="-0.565887 -0.0002 -0.0" rpy="0 0 0"/>
+    <origin xyz="-0.567002 -0.010648 0.015489" rpy="0 0 0"/>
     <geometry>
       <mesh filename="package://HEXAPEDAL_URDF_description/meshes/LM_foot_2_1.stl" scale="0.001 0.001 0.001"/>
@@ -2466,10 +2466,10 @@
 <link name="LB_foot_2_1">
   <inertial>
-    <origin xyz="0.001935898564130012 0.0019356726051708018 0.011535157888886953" rpy="0 0 0"/>
-    <mass value="0.1674566879251433"/>
-    <inertia ixx="3.5e-05" iyy="3.5e-05" izz="5.8e-05" ixy="-1.1e-05" iyz="-0.0" ixz="-0.0"/>
-  </inertial>
-  <visual>
-    <origin xyz="-0.400001 -0.400284 0.0" rpy="0 0 0"/>
+    <origin xyz="0.009349689575527842 -0.005967768422400432 0.0036911038926663777" rpy="0 0 0"/>
+    <mass value="0.1824085742487717"/>
+    <inertia ixx="4.2e-05" iyy="4.2e-05" izz="7e-05" ixy="-1.1e-05" iyz="0.0" ixz="-1e-06"/>
+  </inertial>
+  <visual>
+    <origin xyz="-0.393402 -0.408461 0.015489" rpy="0 0 0"/>
     <geometry>
       <mesh filename="package://HEXAPEDAL_URDF_description/meshes/LB_foot_2_1.stl" scale="0.001 0.001 0.001"/>
@@ -2478,5 +2478,5 @@
   </visual>
   <collision>
-    <origin xyz="-0.400001 -0.400284 0.0" rpy="0 0 0"/>
+    <origin xyz="-0.393402 -0.408461 0.015489" rpy="0 0 0"/>
     <geometry>
       <mesh filename="package://HEXAPEDAL_URDF_description/meshes/LB_foot_2_1.stl" scale="0.001 0.001 0.001"/>
@@ -2486,10 +2486,10 @@
 <link name="RF_foot_2_1">
   <inertial>
-    <origin xyz="-0.001935969016851058 -0.001935295033748785 0.011535187582277775" rpy="0 0 0"/>
-    <mass value="0.1674566879251433"/>
-    <inertia ixx="3.5e-05" iyy="3.5e-05" izz="5.8e-05" ixy="-1.1e-05" iyz="0.0" ixz="0.0"/>
-  </inertial>
-  <visual>
-    <origin xyz="0.400285 0.400001 -0.0" rpy="0 0 0"/>
+    <origin xyz="0.005967768422387609 -0.009349689575525344 -0.0036911038926828853" rpy="0 0 0"/>
+    <mass value="0.1824085742487717"/>
+    <inertia ixx="4.2e-05" iyy="4.2e-05" izz="7e-05" ixy="-1.1e-05" iyz="-1e-06" ixz="0.0"/>
+  </inertial>
+  <visual>
+    <origin xyz="0.408461 0.393402 -0.015489" rpy="0 0 0"/>
     <geometry>
       <mesh filename="package://HEXAPEDAL_URDF_description/meshes/RF_foot_2_1.stl" scale="0.001 0.001 0.001"/>
@@ -2498,5 +2498,5 @@
   </visual>
   <collision>
-    <origin xyz="0.400285 0.400001 -0.0" rpy="0 0 0"/>
+    <origin xyz="0.408461 0.393402 -0.015489" rpy="0 0 0"/>
     <geometry>
       <mesh filename="package://HEXAPEDAL_URDF_description/meshes/RF_foot_2_1.stl" scale="0.001 0.001 0.001"/>
@@ -2506,10 +2506,10 @@
 <link name="RM_foot_2_1">
   <inertial>
-    <origin xyz="-0.002737054550587814 2.9490391404213474e-07 0.011535187582279404" rpy="0 0 0"/>
-    <mass value="0.1674566879251433"/>
-    <inertia ixx="2.4e-05" iyy="4.5e-05" izz="5.8e-05" ixy="0.0" iyz="0.0" ixz="0.0"/>
-  </inertial>
-  <visual>
-    <origin xyz="0.565888 -0.000201 -0.0" rpy="0 0 0"/>
+    <origin xyz="-0.002392144263397622 -0.010830757402981957 -0.003691103892675549" rpy="0 0 0"/>
+    <mass value="0.1824085742487717"/>
+    <inertia ixx="3.1e-05" iyy="5.2e-05" izz="7e-05" ixy="0.0" iyz="-1e-06" ixz="-0.0"/>
+  </inertial>
+  <visual>
+    <origin xyz="0.567002 -0.010648 -0.015489" rpy="0 0 0"/>
     <geometry>
       <mesh filename="package://HEXAPEDAL_URDF_description/meshes/RM_foot_2_1.stl" scale="0.001 0.001 0.001"/>
@@ -2518,5 +2518,5 @@
   </visual>
   <collision>
-    <origin xyz="0.565888 -0.000201 -0.0" rpy="0 0 0"/>
+    <origin xyz="0.567002 -0.010648 -0.015489" rpy="0 0 0"/>
     <geometry>
       <mesh filename="package://HEXAPEDAL_URDF_description/meshes/RM_foot_2_1.stl" scale="0.001 0.001 0.001"/>
@@ -2526,10 +2526,10 @@
 <link name="RB_foot_2_1">
   <inertial>
-    <origin xyz="-0.0019352950337527264 0.0019359690168521126 0.011535187582292222" rpy="0 0 0"/>
-    <mass value="0.1674566879251433"/>
-    <inertia ixx="3.5e-05" iyy="3.5e-05" izz="5.8e-05" ixy="1.1e-05" iyz="-0.0" ixz="0.0"/>
-  </inertial>
-  <visual>
-    <origin xyz="0.400001 -0.400285 -0.0" rpy="0 0 0"/>
+    <origin xyz="-0.009349689575533227 -0.005967768422384057 -0.0036911038926868995" rpy="0 0 0"/>
+    <mass value="0.1824085742487717"/>
+    <inertia ixx="4.2e-05" iyy="4.2e-05" izz="7e-05" ixy="1.1e-05" iyz="-0.0" ixz="-1e-06"/>
+  </inertial>
+  <visual>
+    <origin xyz="0.393402 -0.408461 -0.015489" rpy="0 0 0"/>
     <geometry>
       <mesh filename="package://HEXAPEDAL_URDF_description/meshes/RB_foot_2_1.stl" scale="0.001 0.001 0.001"/>
@@ -2538,5 +2538,5 @@
   </visual>
   <collision>
-    <origin xyz="0.400001 -0.400285 -0.0" rpy="0 0 0"/>
+    <origin xyz="0.393402 -0.408461 -0.015489" rpy="0 0 0"/>
     <geometry>
       <mesh filename="package://HEXAPEDAL_URDF_description/meshes/RB_foot_2_1.stl" scale="0.001 0.001 0.001"/>
@@ -2546,90 +2546,90 @@
 <link name="LF_foot_3_1">
   <inertial>
-    <origin xyz="0.001995229041856117 -0.0019953844862484194 2.7708375447619718e-15" rpy="0 0 0"/>
-    <mass value="0.004532023320514249"/>
+    <origin xyz="0.001072637769902185 -0.0010727950574442868 -2.516513049388941e-13" rpy="0 0 0"/>
+    <mass value="0.0032374522012746203"/>
+    <inertia ixx="0.0" iyy="0.0" izz="0.0" ixy="-0.0" iyz="0.0" ixz="-0.0"/>
+  </inertial>
+  <visual>
+    <origin xyz="-0.425749 0.425466 0.0" rpy="0 0 0"/>
+    <geometry>
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
Commit message: feat(urdf): update Livox model with aligned frame

File: HW/urdf/urdf/HEXAPEDAL_URDF.xacro (robot description, xacro)
@@ -1546,10 +1546,10 @@
 <link name="livox_mid_360_1">
   <inertial>
-    <origin xyz="0.02399969341720557 0.01799971078348498 0.016243790042632766" rpy="3.141592653589793 0 1.5707963267948966"/>
-    <mass value="1.055789101972525"/>
-    <inertia ixx="0.000444" iyy="0.000443" izz="0.000694" ixy="-0.0" iyz="-0.0" ixz="-0.0"/>
-  </inertial>
-  <visual>
-    <origin xyz="0.011962306582794429 0.01792928921651436 0.2746291446897346" rpy="3.141592653589793 0 1.5707963267948966"/>
+    <origin xyz="0.02443105558853103 0.01799971078347508 0.016220816346548705" rpy="3.141592653589793 0 1.5707963267948966"/>
+    <mass value="1.068415791165833"/>
+    <inertia ixx="0.000444" iyy="0.000459" izz="0.000711" ixy="0.0" iyz="-0.0" ixz="1e-06"/>
+  </inertial>
+  <visual>
+    <origin xyz="0.011962306582794464 0.017929289216514384 0.2746291446897346" rpy="3.141592653589793 0 1.5707963267948966"/>
     <geometry>
       <mesh filename="package://HEXAPEDAL_URDF_description/meshes/livox_mid_360_1.stl" scale="0.001 0.001 0.001"/>
@@ -1558,5 +1558,5 @@
   </visual>
   <collision>
-    <origin xyz="0.011962306582794429 0.01792928921651436 0.2746291446897346" rpy="3.141592653589793 0 1.5707963267948966"/>
+    <origin xyz="0.011962306582794464 0.017929289216514384 0.2746291446897346" rpy="3.141592653589793 0 1.5707963267948966"/>
     <geometry>
       <mesh filename="package://HEXAPEDAL_URDF_description/meshes/livox_mid_360_1.stl" scale="0.001 0.001 0.001"/>
