Commit message: Update URDF for revised lidar mount

File: HW/urdf/urdf/HEXAPEDAL_URDF.xacro (robot description, xacro)
@@ -406,5 +406,5 @@
 <link name="RB_flame4_1">
   <inertial>
-    <origin xyz="-0.020163841378833314 0.02016384139333624 -0.0036246185003608977" rpy="0 0 0"/>
+    <origin xyz="-0.020163841378835465 0.020163841393334644 -0.003624618500374904" rpy="0 0 0"/>
     <mass value="0.06395081687871436"/>
     <inertia ixx="6.2e-05" iyy="6.2e-05" izz="7.4e-05" ixy="1.7e-05" iyz="2e-06" ixz="-2e-06"/>
@@ -506,5 +506,5 @@
 <link name="LF_flame4_1">
   <inertial>
-    <origin xyz="0.020163841378835992 -0.020163841393339085 -0.003624618500361524" rpy="0 0 0"/>
+    <origin xyz="0.020163841378832717 -0.020163841393343346 -0.0036246185003829686" rpy="0 0 0"/>
     <mass value="0.06395081687871436"/>
     <inertia ixx="6.2e-05" iyy="6.2e-05" izz="7.4e-05" ixy="1.7e-05" iyz="-2e-06" ixz="2e-06"/>
@@ -526,5 +526,5 @@
 <link name="RF_DS51150_270_1_1">
   <inertial>
-    <origin xyz="-0.023032770266679756 -0.023032770253798393 -0.0067332853591638014" rpy="0 0 0"/>
+    <origin xyz="-0.02303277026668618 -0.023032770253798768 -0.006733285359171658" rpy="0 0 0"/>
     <mass value="0.16496568495572975"/>
     <inertia ixx="6.8e-05" iyy="6.8e-05" izz="7.3e-05" ixy="-2.4e-05" iyz="0.0" ixz="0.0"/>
@@ -566,5 +566,5 @@
 <link name="RB_DS51150_270_1_1">
   <inertial>
-    <origin xyz="-0.023032770253802626 0.023032770266685404 -0.006733285359163047" rpy="0 0 0"/>
+    <origin xyz="-0.02303277025380847 0.023032770266688846 -0.006733285359181024" rpy="0 0 0"/>
     <mass value="0.16496568495572975"/>
     <inertia ixx="6.8e-05" iyy="6.8e-05" izz="7.3e-05" ixy="2.4e-05" iyz="-0.0" ixz="0.0"/>
@@ -586,5 +586,5 @@
 <link name="LF_DS51150_270_1_1">
   <inertial>
-    <origin xyz="0.0230327702538011 -0.02303277026668407 -0.006733285359159725" rpy="0 0 0"/>
+    <origin xyz="0.023032770253793314 -0.023032770266692065 -0.0067332853591978185" rpy="0 0 0"/>
     <mass value="0.16496568495572975"/>
     <inertia ixx="6.8e-05" iyy="6.8e-05" izz="7.3e-05" ixy="2.4e-05" iyz="0.0" ixz="-0.0"/>
@@ -686,5 +686,5 @@
 <link name="RB_bearing_1_1">
   <inertial>
-    <origin xyz="-2.011289298720076e-07 2.0112893012180777e-07 -0.0020000000000093623" rpy="0 0 0"/>
+    <origin xyz="-2.011289320369425e-07 2.0112892845647323e-07 -0.0020000000000233685" rpy="0 0 0"/>
     <mass value="0.003999875766550524"/>
     <inertia ixx="0.0" iyy="0.0" izz="0.0" ixy="0.0" iyz="0.0" ixz="0.0"/>
@@ -706,7 +706,7 @@
 <link name="LF_bearing_1_1">
   <inertial>
-    <origin xyz="2.0112893564516732e-07 -2.0112893614476768e-07 -0.0020000000000144035" rpy="0 0 0"/>
+    <origin xyz="2.0112893234225382e-07 -2.0112894041912632e-07 -0.0020000000000358793" rpy="0 0 0"/>
     <mass value="0.003999875766550524"/>
-    <inertia ixx="0.0" iyy="0.0" izz="0.0" ixy="0.0" iyz="0.0" ixz="-0.0"/>
+    <inertia ixx="0.0" iyy="0.0" izz="0.0" ixy="0.0" iyz="0.0" ixz="0.0"/>
   </inertial>
   <visual>
@@ -984,14 +984,34 @@
   </collision>
 </link>
-<link name="M_column_3_fix_1">
-  <inertial>
-    <origin xyz="-2.8932913603613077e-07 0.0010697115249376009 0.037050770789614454" rpy="0 0 0"/>
-    <mass value="0.4404030088724962"/>
-    <inertia ixx="0.000372" iyy="0.000387" izz="0.000176" ixy="-0.0" iyz="-9e-06" ixz="-0.0"/>
+<link name="제목_없음_1">
+  <inertial>
+    <origin xyz="-0.06208428932188086 -0.033027993162494454 0.013145252856636543" rpy="0 0 0"/>
+    <mass value="0.7007544239040091"/>
+    <inertia ixx="0.00034" iyy="0.003139" izz="0.0034" ixy="-0.0" iyz="1e-06" ixz="0.0"/>
+  </inertial>
+  <visual>
+    <origin xyz="-0.062155 0.062155 -0.0492" rpy="0 0 0"/>
+    <geometry>
+      <mesh filename="package://HEXAPEDAL_URDF_description/meshes/제목_없음_1.stl" scale="0.001 0.001 0.001"/>
+    </geometry>
+    <material name="silver"/>
+  </visual>
+  <collision>
+    <origin xyz="-0.062155 0.062155 -0.0492" rpy="0 0 0"/>
+    <geometry>
+      <mesh filename="package://HEXAPEDAL_URDF_description/meshes/제목_없음_1.stl" scale="0.001 0.001 0.001"/>
+    </geometry>
+  </collision>
+</link>
+<link name="M_column_3_final_1">
+  <inertial>
+    <origin xyz="-2.8927925917434836e-07 0.01867798656025905 0.026383501906955667" rpy="0 0 0"/>
+    <mass value="0.47179646795444613"/>
+    <inertia ixx="0.000375" iyy="0.000291" izz="0.00026" ixy="0.0" iyz="-0.000164" ixz="0.0"/>
   </inertial>
   <visual>
     <origin xyz="-7.1e-05 7.1e-05 -0.0801" rpy="0 0 0"/>
     <geometry>
-      <mesh filename="package://HEXAPEDAL_URDF_description/meshes/M_column_3_fix_1.stl" scale="0.001 0.001 0.001"/>
+      <mesh filename="package://HEXAPEDAL_URDF_description/meshes/M_column_3_final_1.stl" scale="0.001 0.001 0.001"/>
     </geometry>
     <material name="silver"/>
@@ -1000,65 +1020,5 @@
     <origin xyz="-7.1e-05 7.1e-05 -0.0801" rpy="0 0 0"/>
     <geometry>
-      <mesh filename="package://HEXAPEDAL_URDF_description/meshes/M_column_3_fix_1.stl" scale="0.001 0.001 0.001"/>
-    </geometry>
-  </collision>
-</link>
-<link name="livox_mid_360_2">
-  <inertial>
-    <origin xyz="-0.024431329875830785 -0.01799971067812863 -0.016220940752814474" rpy="2.8797932657906444 0 -1.5707963267948966"/>
-    <mass value="1.068415791165833"/>
-    <inertia ixx="0.000459" iyy="0.000462" izz="0.000694" ixy="-0.0" iyz="-6.6e-05" ixz="-0.0"/>
-  </inertial>
-  <visual>
-    <origin xyz="0.012451065790221452 -0.0179292893218819 0.1413104354141189" rpy="2.8797932657906444 0 -1.5707963267948966"/>
-    <geometry>
-      <mesh filename="package://HEXAPEDAL_URDF_description/meshes/livox_mid_360_2.stl" scale="0.001 0.001 0.001"/>
-    </geometry>
-    <material name="silver"/>
-  </visual>
-  <collision>
-    <origin xyz="0.012451065790221452 -0.0179292893218819 0.1413104354141189" rpy="2.8797932657906444 0 -1.5707963267948966"/>
-    <geometry>
-      <mesh filename="package://HEXAPEDAL_URDF_description/meshes/livox_mid_360_2.stl" scale="0.001 0.001 0.001"/>
-    </geometry>
-  </collision>
-</link>
-<link name="camera_fixer_1">
-  <inertial>
-    <origin xyz="-0.011000279135611947 -0.005377992721875585 -0.001403699933637606" rpy="0 0 0"/>
-    <mass value="0.10205435536884809"/>
-    <inertia ixx="9e-06" iyy="1.7e-05" izz="1.7e-05" ixy="-0.0" iyz="0.0" ixz="0.0"/>
-  </inertial>
-  <visual>
-    <origin xyz="-0.011071 0.009071 -0.1161" rpy="0 0 0"/>
-    <geometry>
-      <mesh filename="package://HEXAPEDAL_URDF_description/meshes/camera_fixer_1.stl" scale="0.001 0.001 0.001"/>
-    </geometry>
-    <material name="silver"/>
-  </visual>
-  <collision>
-    <origin xyz="-0.011071 0.009071 -0.1161" rpy="0 0 0"/>
-    <geometry>
-      <mesh filename="package://HEXAPEDAL_URDF_description/meshes/camera_fixer_1.stl" scale="0.001 0.001 0.001"/>
-    </geometry>
-  </collision>
-</link>
-<link name="mid-360-fov-asm_ver.ksh_MID-360_4_1_1_1">
-  <inertial>
-    <origin xyz="-3.0009021704220456e-07 -0.002702514686128593 0.010087666111087745" rpy="0 0 0"/>
-    <mass value="0.2760142598595122"/>
-    <inertia ixx="4.7e-05" iyy="4.8e-05" izz="6.5e-05" ixy="-0.0" iyz="-5e-06" ixz="-0.0"/>
-  </inertial>
-  <visual>
-    <origin xyz="-7.1e-05 0.010436 -0.179782" rpy="0 0 0"/>
-    <geometry>
-      <mesh filename="package://HEXAPEDAL_URDF_description/meshes/mid-360-fov-asm_ver.ksh_MID-360_4_1_1_1.stl" scale="0.001 0.001 0.001"/>
-    </geometry>
-    <material name="silver"/>
-  </visual>
-  <collision>
-    <origin xyz="-7.1e-05 0.010436 -0.179782" rpy="0 0 0"/>
-    <geometry>
-      <mesh filename="package://HEXAPEDAL_URDF_description/meshes/mid-360-fov-asm_ver.ksh_MID-360_4_1_1_1.stl" scale="0.001 0.001 0.001"/>
+      <mesh filename="package://HEXAPEDAL_URDF_description/meshes/M_column_3_final_1.stl" scale="0.001 0.001 0.001"/>
     </geometry>
   </collision>
@@ -1066,5 +1026,5 @@
 <link name="LF_motor_horn_1_1">
   <inertial>
-    <origin xyz="2.0112883633571776e-07 -2.0112900966928748e-07 -0.0029620014635887496" rpy="0 0 0"/>
+    <origin xyz="2.0112882836986756e-07 -2.0112901788493787e-07 -0.0029620014636270384" rpy="0 0 0"/>
     <mass value="0.0019994583976964877"/>
     <inertia ixx="0.0" iyy="0.0" izz="0.0" ixy="0.0" iyz="-0.0" ixz="-0.0"/>
@@ -1106,5 +1066,5 @@
 <link name="LB_motor_horn_1_1">
   <inertial>
-    <origin xyz="2.0112900539492884e-07 2.0112883239442603e-07 -0.002962001463592448" rpy="0 0 0"/>
+    <origin xyz="2.011290100023544e-07 2.0112882784251163e-07 -0.0029620014636008683" rpy="0 0 0"/>
     <mass value="0.0019994583976964877"/>
     <inertia ixx="0.0" iyy="0.0" izz="0.0" ixy="-0.0" iyz="-0.0" ixz="0.0"/>
@@ -1166,5 +1126,5 @@
 <link name="RB_motor_horn_1_1">
   <inertial>
-    <origin xyz="-2.0112883974965357e-07 2.0112901288893426e-07 -0.0029620014635853113" rpy="0 0 0"/>
+    <origin xyz="-2.0112884444034584e-07 2.0112901552571394e-07 -0.0029620014636034253" rpy="0 0 0"/>
     <mass value="0.0019994583976964877"/>
     <inertia ixx="0.0" iyy="0.0" izz="0.0" ixy="0.0" iyz="0.0" ixz="0.0"/>
@@ -1206,5 +1166,5 @@
 <link name="RM_coxaR_1">
   <inertial>
-    <origin xyz="-0.037000000855337584 0.0004226038534422383 -0.03422260266699357" rpy="0 0 0"/>
+    <origin xyz="-0.03700000085533775 0.00042260385343186437 -0.034222602666993715" rpy="0 0 0"/>
     <mass value="0.09366200268610271"/>
     <inertia ixx="0.000108" iyy="0.000126" izz="0.000126" ixy="1e-06" iyz="-0.0" ixz="1e-06"/>
@@ -1226,5 +1186,5 @@
 <link name="RB_coxaR_1">
   <inertial>
-    <origin xyz="-0.025864326587123065 0.02646197868816627 -0.034222602666985784" rpy="0 0 0"/>
+    <origin xyz="-0.025864326587127562 0.026461978688168936 -0.034222602667003915" rpy="0 0 0"/>
     <mass value="0.09366200268610271"/>
     <inertia ixx="0.000118" iyy="0.000115" izz="0.000126" ixy="9e-06" iyz="-1e-06" ixz="1e-06"/>
@@ -1246,5 +1206,5 @@
 <link name="LF_coxaL_1">
   <inertial>
-    <origin xyz="0.026461977339774206 -0.02586432793551094 -0.0342226026670027" rpy="0 0 0"/>
+    <origin xyz="0.026461977339766296 -0.0258643279355191 -0.03422260266704109" rpy="0 0 0"/>
     <mass value="0.09366200268610271"/>
     <inertia ixx="0.000115" iyy="0.000118" izz="0.000126" ixy="9e-06" iyz="1e-06" ixz="-1e-06"/>
@@ -1286,5 +1246,5 @@
 <link name="LB_coxaL_1">
   <inertial>
-    <origin xyz="0.025864327935505804 0.026461977339768905 -0.03422260266700408" rpy="0 0 0"/>
+    <origin xyz="0.02586432793551041 0.026461977339764214 -0.0342226026670124" rpy="0 0 0"/>
     <mass value="0.09366200268610271"/>
     <inertia ixx="0.000118" iyy="0.000115" izz="0.000126" ixy="-9e-06" iyz="-1e-06" ixz="-1e-06"/>
@@ -1326,5 +1286,5 @@
 <link name="RM_motor_horn_2_1">
   <inertial>
-    <origin xyz="-1.2212453270876722e-15 0.003862001463596998 -1.2308238216877004e-13" rpy="0 0 0"/>
+    <origin xyz="2.7755575615628914e-16 0.00386200146358686 -1.2329364841068194e-13" rpy="0 0 0"/>
     <mass value="0.0019994583976964877"/>
     <inertia ixx="0.0" iyy="0.0" izz="0.0" ixy="0.0" iyz="0.0" ixz="-0.0"/>
@@ -1346,10 +1306,10 @@
 <link name="RB_motor_horn_2_1">
   <inertial>
-    <origin xyz="0.0027305352830218066 0.002730741156485167 -1.1531083698720926e-13" rpy="0 0 0"/>
+    <origin xyz="0.0027305352830171714 0.002730741156487887 -1.3337612854330877e-13" rpy="0 0 0"/>
     <mass value="0.0019994583976964877"/>
     <inertia ixx="0.0" iyy="0.0" izz="0.0" ixy="0.0" iyz="0.0" ixz="0.0"/>
   </inertial>
   <visual>
-    <origin xyz="0.206687 -0.158887 -0.0" rpy="0 0 0"/>
+    <origin xyz="0.206687 -0.158887 0.0" rpy="0 0 0"/>
     <geometry>
       <mesh filename="package://HEXAPEDAL_URDF_description/meshes/RB_motor_horn_2_1.stl" scale="0.001 0.001 0.001"/>
@@ -1358,5 +1318,5 @@
   </visual>
   <collision>
-    <origin xyz="0.206687 -0.158887 -0.0" rpy="0 0 0"/>
+    <origin xyz="0.206687 -0.158887 0.0" rpy="0 0 0"/>
     <geometry>
       <mesh filename="package://HEXAPEDAL_URDF_description/meshes/RB_motor_horn_2_1.stl" scale="0.001 0.001 0.001"/>
@@ -1366,10 +1326,10 @@
 <link name="LF_motor_horn_2_1">
   <inertial>
-    <origin xyz="0.0027307411564834183 0.0027305352830214458 1.2307251773562983e-13" rpy="0 0 0"/>
+    <origin xyz="0.002730741156475508 0.002730535283013563 8.548115031890303e-14" rpy="0 0 0"/>
     <mass value="0.0019994583976964877"/>
     <inertia ixx="0.0" iyy="0.0" izz="0.0" ixy="0.0" iyz="-0.0" ixz="-0.0"/>
   </inertial>
   <visual>
-    <origin xyz="-0.158887 0.206687 -0.0" rpy="0 0 0"/>
+    <origin xyz="-0.158887 0.206687 0.0" rpy="0 0 0"/>
     <geometry>
       <mesh filename="package://HEXAPEDAL_URDF_description/meshes/LF_motor_horn_2_1.stl" scale="0.001 0.001 0.001"/>
@@ -1378,5 +1338,5 @@
   </visual>
   <collision>
-    <origin xyz="-0.158887 0.206687 -0.0" rpy="0 0 0"/>
+    <origin xyz="-0.158887 0.206687 0.0" rpy="0 0 0"/>
     <geometry>
       <mesh filename="package://HEXAPEDAL_URDF_description/meshes/LF_motor_horn_2_1.stl" scale="0.001 0.001 0.001"/>
@@ -1406,5 +1366,5 @@
 <link name="LB_motor_horn_2_1">
   <inertial>
-    <origin xyz="-0.0027305352830285234 0.002730741156477867 1.216963209818856e-13" rpy="0 0 0"/>
+    <origin xyz="-0.0027305352830239438 0.0027307411564732598 1.1333888079242351e-13" rpy="0 0 0"/>
     <mass value="0.0019994583976964877"/>
     <inertia ixx="0.0" iyy="0.0" izz="0.0" ixy="-0.0" iyz="-0.0" ixz="0.0"/>
@@ -1426,10 +1386,10 @@
 <link name="LF_DS51150_270_2_1">
   <inertial>
-    <origin xyz="0.03560985654621959 0.008136788935394268 9.110513602833456e-12" rpy="0 0 0"/>
+    <origin xyz="0.03560985654621199 0.008136788935386469 9.072852876170052e-12" rpy="0 0 0"/>
     <mass value="0.16496568495572975"/>
     <inertia ixx="5.8e-05" iyy="5.9e-05" izz="9.3e-05" ixy="1.5e-05" iyz="0.0" ixz="0.0"/>
   </inertial>
   <visual>
-    <origin xyz="-0.159523 0.206051 -0.0" rpy="0 0 0"/>
+    <origin xyz="-0.159523 0.206051 0.0" rpy="0 0 0"/>
     <geometry>
       <mesh filename="package://HEXAPEDAL_URDF_description/meshes/LF_DS51150_270_2_1.stl" scale="0.001 0.001 0.001"/>
@@ -1438,5 +1398,5 @@
   </visual>
   <collision>
-    <origin xyz="-0.159523 0.206051 -0.0" rpy="0 0 0"/>
+    <origin xyz="-0.159523 0.206051 0.0" rpy="0 0 0"/>
     <geometry>
       <mesh filename="package://HEXAPEDAL_URDF_description/meshes/LF_DS51150_270_2_1.stl" scale="0.001 0.001 0.001"/>
@@ -1466,5 +1426,5 @@
 <link name="LB_DS51150_270_2_1">
   <inertial>
-    <origin xyz="-0.008136788935400124 0.03560985654621082 9.108673217267947e-12" rpy="0 0 0"/>
+    <origin xyz="-0.008136788935395461 0.03560985654620624 9.100279146254787e-12" rpy="0 0 0"/>
     <mass value="0.16496568495572975"/>
     <inertia ixx="5.9e-05" iyy="5.8e-05" izz="9.3e-05" ixy="-1.5e-05" iyz="0.0" ixz="-0.0"/>
@@ -1506,5 +1466,5 @@
 <link name="RM_DS51150_270_2_1">
   <inertial>
-    <origin xyz="-0.01942624683308497 0.03093328535917127 -9.111592340665953e-12" rpy="0 0 0"/>
+    <origin xyz="-0.019426246833087912 0.03093328535915816 -9.10996944823753e-12" rpy="0 0 0"/>
     <mass value="0.16496568495572975"/>
     <inertia ixx="4.4e-05" iyy="7.3e-05" izz="9.3e-05" ixy="0.0" iyz="-0.0" ixz="-0.0"/>
@@ -1526,10 +1486,10 @@
 <link name="RB_DS51150_270_2_1">
   <inertial>
-    <origin xyz="0.00813678893539413 0.03560985654621854 -9.102308010916462e-12" rpy="0 0 0"/>
+    <origin xyz="0.0081367889353893 0.035609856546221175 -9.120399476032414e-12" rpy="0 0 0"/>
     <mass value="0.16496568495572975"/>
     <inertia ixx="5.9e-05" iyy="5.8e-05" izz="9.3e-05" ixy="1.5e-05" iyz="-0.0" ixz="-0.0"/>
   </inertial>
   <visual>
-    <origin xyz="0.206051 -0.159523 -0.0" rpy="0 0 0"/>
+    <origin xyz="0.206051 -0.159523 0.0" rpy="0 0 0"/>
     <geometry>
       <mesh filename="package://HEXAPEDAL_URDF_description/meshes/RB_DS51150_270_2_1.stl" scale="0.001 0.001 0.001"/>
@@ -1538,5 +1498,5 @@
   </visual>
   <collision>
-    <origin xyz="0.206051 -0.159523 -0.0" rpy="0 0 0"/>
+    <origin xyz="0.206051 -0.159523 0.0" rpy="0 0 0"/>
     <geometry>
       <mesh filename="package://HEXAPEDAL_URDF_description/meshes/RB_DS51150_270_2_1.stl" scale="0.001 0.001 0.001"/>
@@ -1544,7 +1504,27 @@
   </collision>
 </link>
+<link name="livox_mid_360_2">
+  <inertial>
+    <origin xyz="-0.0235686244929285 0.017999710678128677 -0.01622143724251992" rpy="2.3561944901923453 0 1.5707963267948966"/>
+    <mass value="1.068415791165833"/>
+    <inertia ixx="0.000459" iyy="0.000577" izz="0.000579" ixy="-0.0" iyz="-0.000134" ixz="-0.0"/>
+  </inertial>
+  <visual>
+    <origin xyz="-0.14005665348536553 0.017929289321881845 0.06915693361984346" rpy="2.3561944901923453 0 1.5707963267948966"/>
+    <geometry>
+      <mesh filename="package://HEXAPEDAL_URDF_description/meshes/livox_mid_360_2.stl" scale="0.001 0.001 0.001"/>
+    </geometry>
+    <material name="silver"/>
+  </visual>
+  <collision>
+    <origin xyz="-0.14005665348536553 0.017929289321881845 0.06915693361984346" rpy="2.3561944901923453 0 1.5707963267948966"/>
+    <geometry>
+      <mesh filename="package://HEXAPEDAL_URDF_description/meshes/livox_mid_360_2.stl" scale="0.001 0.001 0.001"/>
+    </geometry>
+  </collision>
+</link>
 <link name="RF_link1_right_1">
   <inertial>
-    <origin xyz="-0.022677020519566077 -0.037455160000820775 -0.015609126867096363" rpy="0 0 0"/>
+    <origin xyz="-0.022677021050098972 -0.03745516077457217 -0.015609126867096599" rpy="0 0 0"/>
     <mass value="0.05250233789665554"/>
     <inertia ixx="6.3e-05" iyy="6.3e-05" izz="0.000106" ixy="-4.5e-05" iyz="-1e-06" ixz="1e-06"/>
@@ -1566,5 +1546,5 @@
 <link name="RF_DS51150_270_3_1">
   <inertial>
-    <origin xyz="0.017106763843891093 -0.017211590398439225 -0.014999999990897343" rpy="0 0 0"/>
+    <origin xyz="0.017106763797174407 -0.017211590721209924 -0.01499999999089773" rpy="0 0 0"/>
     <mass value="0.16496568495572975"/>
     <inertia ixx="5.9e-05" iyy="5.8e-05" izz="9.3e-05" ixy="-1.5e-05" iyz="0.0" ixz="-0.0"/>
@@ -1586,5 +1566,5 @@
 <link name="RF_bearing_2_1">
   <inertial>
-    <origin xyz="-0.0014145438679431521 0.001413913558223956 -7.574574939285309e-15" rpy="0 0 0"/>
+    <origin xyz="-0.0014145445240567045 0.0014139128534798595 -7.793169765454425e-15" rpy="0 0 0"/>
     <mass value="0.003999875766550524"/>
     <inertia ixx="0.0" iyy="0.0" izz="0.0" ixy="-0.0" iyz="0.0" ixz="0.0"/>
@@ -1606,5 +1586,5 @@
 <link name="RF_bearing_3_1">
   <inertial>
-    <origin xyz="-0.001414573372445882 0.0014138844492528058 -6.518651033802115e-15" rpy="0 0 0"/>
+    <origin xyz="-0.00141457383079302 0.0014138835467424338 -6.671790675630351e-15" rpy="0 0 0"/>
     <mass value="0.003999875766550524"/>
     <inertia ixx="0.0" iyy="0.0" izz="0.0" ixy="-0.0" iyz="0.0" ixz="-0.0"/>
@@ -1626,5 +1606,5 @@
 <link name="RM_link1_right_1">
   <inertial>
-    <origin xyz="-0.04251961074375388 -0.010449696082231551 -0.015609126867089297" rpy="0 0 0"/>
+    <origin xyz="-0.04251961166602958 -0.010449696254225434 -0.01560912686708989" rpy="0 0 0"/>
     <mass value="0.05250233789665554"/>
     <inertia ixx="1.8e-05" iyy="0.000108" izz="0.000106" ixy="0.0" iyz="-1e-06" ixz="0.0"/>
@@ -1646,5 +1626,5 @@
 <link name="RM_DS51150_270_3_1">
   <inertial>
-    <origin xyz="-7.375365070272366e-05 -0.02426671444562294 -0.014999999990891844" rpy="0 0 0"/>
+    <origin xyz="-7.375391196973169e-05 -0.02426671464084055 -0.014999999990891074" rpy="0 0 0"/>
     <mass value="0.16496568495572975"/>
     <inertia ixx="4.4e-05" iyy="7.3e-05" izz="9.3e-05" ixy="-0.0" iyz="0.0" ixz="-0.0"/>
@@ -1666,5 +1646,5 @@
 <link name="RM_bearing_2_1">
   <inertial>
-    <origin xyz="1.9010540919239816e-09 0.0020000000343882787 -3.9356945040852597e-16" rpy="0 0 0"/>
+    <origin xyz="9.387737254229478e-10 0.0019999999999936666 -9.936434388075706e-16" rpy="0 0 0"/>
     <mass value="0.003999875766550524"/>
     <inertia ixx="0.0" iyy="0.0" izz="0.0" ixy="0.0" iyz="0.0" ixz="-0.0"/>
@@ -1686,249 +1666,249 @@
 <link name="RM_bearing_3_1">
   <inertial>
-    <origin xyz="-9.301727721400255e-10 0.0020000003140845067 -2.076281183175288e-15" rpy="0 0 0"/>
+    <origin xyz="-1.89244730997018e-09 0.0019999999999949607 3.74119312038047e-17" rpy="0 0 0"/>
+    <mass value="0.003999875766550524"/>
+    <inertia ixx="0.0" iyy="0.0" izz="0.0" ixy="-0.0" iyz="0.0" ixz="-0.0"/>
+  </inertial>
+  <visual>
+    <origin xyz="0.3825 -0.0273 -0.0" rpy="0 0 0"/>
+    <geometry>
+      <mesh filename="package://HEXAPEDAL_URDF_description/meshes/RM_bearing_3_1.stl" scale="0.001 0.001 0.001"/>
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